Commit message: add ball, kp=20 for smoothness, dr and noise for real, trained planner and height estimator with imitation

File: legged_gym/resources/robots/ball.urdf (robot description, URDF)
Before this commit: robot ball, 1 links, 0 joints
Links:
- link ball: mass 0.5 -> 10; geometry collision sphere radius=0.17; visual sphere radius=0.17
