Commit message: modify the ppo alg and replay buffer for training seperate mode

File: legged_gym/resources/robots/go1/urdf/go1.urdf (robot description, URDF)
Before this commit: robot go1, 34 links, 33 joints
Joints:
- joint 1_FR_thigh_joint: limit lower=-0.686 upper=4.501 effort=23.7 velocity=30.1 -> lower=-0.686 upper=3.92 effort=23.7 velocity=30.1
- joint 2_FL_thigh_joint: limit lower=-0.686 upper=4.501 effort=23.7 velocity=30.1 -> lower=-0.686 upper=3.92 effort=23.7 velocity=30.1

File: legged_gym/resources/robots/go1/urdf/go1_arrow.urdf (robot description, URDF)
Before this commit: robot go1, 35 links, 34 joints
Joints:
- joint 1_FR_thigh_joint: limit lower=-0.686 upper=4.501 effort=23.7 velocity=30.1 -> lower=-0.686 upper=3.92 effort=23.7 velocity=30.1
- joint 2_FL_thigh_joint: limit lower=-0.686 upper=4.501 effort=23.7 velocity=30.1 -> lower=-0.686 upper=3.92 effort=23.7 velocity=30.1
